File: hardware/ffp.kicad_pcb (KiCad board)
At the start: 2 copper layers, 41.3 x 10.7 mm, 17 parts, among them IC1 STM32F042K6T7, IC2 MCP1700, IC3 MIC2004-0_5YM5, J2 USB_C_Receptacle_USB2.0, J3 PROG, P1 SWD_TC

Commit message: replated copper to the top and updated gerber files
Routing:
- added copper zone on F.Cu, net GND
Changed lines of the file:
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@@
+    )
+  )
+  (zone (net 0) (net_name "") (layer F.Cu) (hatch edge 0.508)
+    (connect_pads (clearance 0.275))
+    (min_thickness 0.254)
+    (keepout (tracks allowed) (vias allowed) (copperpour not_allowed))
+    (fill (arc_segments 32) (thermal_gap 0.508) (thermal_bridge_width 0.508))
+    (polygon
+      (pts
+        (xy 120.50014 121.00052) (xy 127.50038 121.00052) (xy 127.50038 124.99848) (xy 120.50014 124.99848)
+      )
+    )
+  )
+  (zone (net 1) (net_name GND) (layer F.Cu) (hatch edge 0.508)
+    (connect_pads (clearance 0.275))
+    (min_thickness 0.254)
+    (fill yes (arc_segments 32) (thermal_gap 0.275) (thermal_bridge_width 0.275))
+    (polygon
+      (pts
+        (xy 111.87684 114.17046) (xy 154.27706 114.17046) (xy 154.27706 126.00686) (xy 111.87684 126.00686)
+      )
     )
   )

Commit message: replaced the connector with a dual row 5pin header with 1.27mm pitch
Parts:
- J3: footprint agg:FTSH-105-01-L-DV-K -> Connector_PinHeader_1.27mm:PinHeader_2x05_P1.27mm_Vertical
- moved J3 2.61 mm to (150.6, 122.5), turned to 180 degrees
Routing:
- net GND: track 37.1 -> 26.0 mm, vias 14 -> 12
- net /SCK: track 17.6 -> 19.0 mm
- net /FPGA_~RST: track 15.2 -> 16.6 mm
- net /FLASH_~CS: track 13.4 -> 14.8 mm
- net /FLASH_SI: track 24.7 -> 26.2 mm
- net /FLASH_SO: track 24.3 -> 25.6 mm
Other:
- board text added: "FFP Rev 1.0"
- board text removed: "Flash/FPGA Programmer Rev 1.0"
