File: hardware/ffp.sch (KiCad schematic (older format))
At the start: 17 parts, among them IC1 STM32F042K6T7, IC2 MCP1700, IC3 MIC2004-0_5YM5, J2 USB_C_Receptacle_USB2.0, J3 PROG, P1 SWD_TC

Commit message: replaced the connector with a dual row 5pin header with 1.27mm pitch
Parts:
- J3: footprint agg:FTSH-105-01-L-DV-K -> Connector_PinHeader_1.27mm:PinHeader_2x05_P1.27mm_Vertical
Changed lines of the file:
@@
 F 0 "J3" H 6600 4915 50  0000 C CNN
 F 1 "PROG" H 6600 4824 50  0000 C CNN
-F 2 "agg:FTSH-105-01-L-DV-K" H 6650 4700 50  0001 C CNN
+F 2 "Connector_PinHeader_1.27mm:PinHeader_2x05_P1.27mm_Vertical" H 6650 4700 50  0001 C CNN
 F 3 "" H 6650 4700 50  0001 C CNN
 F 4 "2856437" H 6650 4700 50  0001 C CNN "Farnell"
